File: XYZ_control/XYZ_board/XYZboard.kicad_pcb (KiCad board)
At the start: 4 copper layers, 127 x 45.7 mm, 75 parts, among them J1 DB9 X, J10 DB9 Y, J11 Gnd Out, J12 Sensor X, J13 Sensor Y, J14 Sensor Z, J15 DB9 Z, J2 Control X, J3 Control Y, J4 Control Z, J5 PWR IN, J6 Settings X, J7 Settings Y, J8 Settings Z, J9 Vcc Out, U1 LM317MSTT3G_Voltage_Regulator, U2 A4988_stepper_driver, U3 A4988_stepper_driver, U4 A4988_stepper_driver

Commit message: xyz board progress
Parts:
- moved C20 63.4 mm to (193.0, 60.3), turned to 270 degrees
- moved C17 63.1 mm to (96.9, 60.4), turned to 270 degrees
- moved C16 56.2 mm to (106.4, 60.4), turned to 270 degrees
- moved C19 56.1 mm to (182.9, 60.3), turned to 270 degrees
- moved R2 48.9 mm to (123.2, 76.2)
- moved LED1 48.0 mm to (123.2, 81.5)
- moved C4 47.8 mm to (119.1, 76.2)
- moved U1 44.4 mm to (165.1, 58.4), turned to 0 degrees
- moved C18 41.4 mm to (149.6, 60.4), turned to 270 degrees
- moved C21 39.9 mm to (122.9, 68.1), turned to 90 degrees
- moved D1 38.9 mm to (83.8, 66.0), turned to 90 degrees
- moved J14 29.0 mm to (175.3, 88.9)
- moved R8 28.4 mm to (176.5, 81.3)
- moved R9 28.4 mm to (174.0, 81.3)
- moved C3 24.7 mm to (192.0, 73.7)
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Connections:
- RA3 pad 3: dir3 -> step3
- RA3 pad 4: step3 -> dir3
Routing:
- net V+: track 0.00 -> 233.2 mm, vias 0 -> 21
- net GND: track 36.1 -> 129.8 mm, vias 11 -> 38
- net sensor2_3: track 0.00 -> 54.3 mm
- net sensor2_2: track 0.00 -> 54.3 mm
- net sensor1_3: track 0.00 -> 49.3 mm
- net sensor1_2: track 0.00 -> 49.2 mm
- net VCC: track 19.0 -> 64.3 mm, vias 8 -> 24
- net dir2: track 0.00 -> 32.4 mm, vias 0 -> 4
- net dir3: track 0.00 -> 31.3 mm, vias 0 -> 2
- net enable3: track 0.00 -> 31.3 mm, vias 0 -> 2
- net enable2: track 0.00 -> 29.3 mm, vias 0 -> 2
- net step3: track 0.00 -> 28.9 mm, vias 0 -> 2
- net step2: track 0.00 -> 28.4 mm, vias 0 -> 2
- net ms2_2: track 0.00 -> 25.4 mm, vias 0 -> 2
- net ms1_3: track 0.00 -> 24.5 mm, vias 0 -> 2
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- added copper zone on F.Cu, net VCC
- removed copper zone on F.Cu, net GND
Other:
- board text added: "CONTROL"
- board text added: "DIR"
- board text added: "ENABLE"
- board text added: "END"
- board text added: "ENDSTOPS"
- board text added: "HOME"
- board text added: "MS1"
- board text added: "MS2"
- board text added: "MS3"
- board text added: "RESET"
- board text added: "SETTINGS"
- board text added: "SLEEP"
- board text added: "STEP"

Commit message: Updated the board and added output files
Parts:
- added mounting hole0_13: VAL**, XYZ_footprints:mounting_hole_0_13_in, F.Cu at (166.4, 87.6)
- added mounting hole0_13: VAL**, XYZ_footprints:mounting_hole_0_13_in, F.Cu at (123.2, 49.5)
- added mounting hole0_13: VAL**, XYZ_footprints:mounting_hole_0_13_in, F.Cu at (123.2, 87.6)
- added mounting hole0_13: VAL**, XYZ_footprints:mounting_hole_0_13_in, F.Cu at (166.4, 49.5)
- added mounting hole0_13: VAL**, XYZ_footprints:mounting_hole_0_13_in, F.Cu at (204.5, 80.0)
- added mounting hole0_13: VAL**, XYZ_footprints:mounting_hole_0_13_in, F.Cu at (85.1, 81.3)
- moved R5 1.58 mm to (90.2, 81.3)
- moved R4 1.58 mm to (92.7, 81.3)
Routing:
- net VCC: track 64.3 -> 63.3 mm
Other:
- board text added: "For Trimpot Adjustment: Vref = Imotor * 8 * .11"
- board text added: "GND"
- board text added: "Gnd"
- board text added: "VCC"
- board text added: "Vin"
