File: AnalogReceiver/KiCad/AmpFil/AmpFil.kicad_pcb (KiCad board)
At the start: 2 copper layers, 43 parts, among them P1 CONN_01X02, P2 CONN_01X02, P3 CONN_01X02, P4 CONN_02X03, P5 CONN_01X02, P6 CONN_01X02, P7 CONN_01X02, U1 SiPM, U2 LT1677, U3 LT1677, U4 LT1677, U5 LT1677

Commit message: Last changes
I made some last changes to the PCB, mainly bias.
Routing:
- net /A2: track 30.6 -> 31.6 mm
