File: High Voltage/Kicad/Parent Folder.kicad_pcb (KiCad board)
At the start: 2 copper layers, 61 parts, among them Q1 STN0214, Q2 STN0214, Q3 STN0214, Q4 BUT11A, Q5 NPN, U1 OP275, U2 OP275, U3 TEENSY3.1, U4 EMCO_F40

Commit message: Made a few changes to the board. I think it's ready to be milled
Parts:
- added REF**: MountingHole_3mm, Mounting_Holes:MountingHole_3mm, F.Cu at (9.14, 44.2)
- added REF**: MountingHole_2-5mm, Mounting_Holes:MountingHole_2-5mm, F.Cu at (26.9, 166.1)
- added REF**: MountingHole_2-5mm, Mounting_Holes:MountingHole_2-5mm, F.Cu at (153.4, 166.1)
- added REF**: , Mounting_Holes:MountingHole_2-5mm, F.Cu at (153.4, 37.1)
- added REF**: , Mounting_Holes:MountingHole_2-5mm, F.Cu at (26.9, 37.1)
- added TP14: GND, Connect:PINTST, F.Cu at (129.5, 88.9)
- added TP15: GND, Connect:PINTST, F.Cu at (132.1, 88.9)
- added TP16: +12V, Connect:PINTST, F.Cu at (96.5, 108.2)
- added TP17: +12V, Connect:PINTST, F.Cu at (98.0, 140.7)
- added TP18: +12V, Connect:PINTST, F.Cu at (93.0, 144.3)
- added TP19: -12V, Connect:PINTST, F.Cu at (117.9, 108.2)
- added TP20: -12V, Connect:PINTST, F.Cu at (116.8, 144.3)
- added TP21: -12V, Connect:PINTST, F.Cu at (119.4, 141.7)
- added TP22: +5V, Connect:PINTST, F.Cu at (134.1, 140.7)
- Q4: value BUT11A -> TIPXXX
- R31: value Varable_Res -> POT
- TP1, TP13, TP2, TP4: value Test_point -> TP
- TP10: value Test_point -> A0
- TP11, TP12, TP5: value Test_point -> (none)
- TP8: value Test_point -> A1
- moved R7 6.49 mm to (105.4, 116.8)
- moved R3 6.35 mm to (110.3, 119.0)
- moved U2 2.54 mm to (105.4, 111.8)
- moved R6 0.78 mm to (108.0, 132.1)
- moved Q4 0.45 mm to (96.5, 99.1)
- moved R2 0.22 mm to (113.0, 129.5)
Routing:
- net GND: track 108.7 -> 582.1 mm
- net +12V: track 8.51 -> 33.7 mm
- net -12V: track 0.00 -> 15.2 mm
- net Net-(R3-Pad2): track 19.2 -> 9.52 mm
- net Net-(R21-Pad1): track 0.00 -> 7.38 mm
- net Net-(Q2-Pad2): track 30.4 -> 24.9 mm
- net Net-(Q1-Pad2): track 30.7 -> 25.1 mm
- net +5V: track 0.00 -> 5.30 mm
- net Net-(Q3-Pad2): track 30.4 -> 26.1 mm
- net Net-(R12-Pad2): track 9.40 -> 12.6 mm
- net Net-(R5-Pad1): track 30.4 -> 33.4 mm
- net Net-(U2-Pad3): track 25.8 -> 23.3 mm
- net Net-(R4-Pad2): track 9.68 -> 12.2 mm
- net Net-(R11-Pad2): track 30.0 -> 32.0 mm
- net Net-(R1-Pad2): track 10.9 -> 12.3 mm
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- added copper zone on B.Cu, net (none)
Other:
- board outline added: 134.6 x 137.2 mm
- net class GND added: clearance 0.5, trace_width 0.4, via_dia 0.889, via_drill 0.635
- net class HV added: clearance 0.5, trace_width 1.5, via_dia 0.889, via_drill 0.635

Commit message: Additional changes to the board, drill files, etc
Parts:
- removed the REF** at (9.14, 44.2)
- Q4: value TIPXXX -> BUT11A
- R31: value POT -> Varable_Res
- REF** (x2): value MountingHole_2-5mm -> (none)
- TP1, TP13, TP2, TP4: value TP -> Test_point
- TP10: value A0 -> Test_point
- TP11, TP12, TP5: value (none) -> Test_point
- TP14, TP15: value GND -> Test_point
- TP16, TP17, TP18: value +12V -> Test_point
- TP19, TP20, TP21: value -12V -> Test_point
- TP22: value +5V -> Test_point
- TP8: value A1 -> Test_point
Routing:
- net GND: track 582.1 -> 555.1 mm
- net +12V: track 33.7 -> 34.6 mm
Other:
- net class Default: clearance 0.254 -> 0.3; trace_width 0.254 -> 0.3
- net class GND: clearance 0.5 -> 1; trace_width 0.4 -> 1
- net class HV: clearance 0.5 -> 1
- net class PowerIn added: clearance 0.7, trace_width 1, via_dia 0.889, via_drill 0.635
- rule trace_clearance: 0.254 -> 0.3
