File: Analog/AnalogReceiver_v2/KiCad/AmpFil/AmpFil.sch (KiCad schematic (older format))
At the start: 49 parts, among them P1 CONN_01X02, P10 CONN_01X02, P11 CONN_01X02, P2 CONN_01X02, P3 CONN_01X02, P4 CONN_01X02, P5 CONN_01X02, P6 CONN_01X02, P7 CONN_01X02, P8 CONN_01X02, P9 CONN_01X02, U1 LT1677, U2 SiPM, U3 LT1677, U4 LT1677, U5 LT1677

Commit message: Updating Files
Making sure all files are up to date for the project documentation.
Parts:
- C2: value 22n -> 15n
- C4, C5: value 33n -> 3.3n
- C6: value 22n -> 47n
- C8: value 10n -> 22n
- R10, R9: value 480k -> 660k
- R11: value 15k -> 8.2k
- R12: value 11k -> 8.2k
- R13: value 120k -> 100k
- R14: value 33k -> 27k
- R5: value 12k -> 10k
- R8: value 4.7k -> 3.9k
Changed lines of the file:
@@
 P 2250 2550
 F 0 "R5" V 2330 2550 50  0000 C CNN
-F 1 "12k" V 2257 2551 50  0000 C CNN
+F 1 "10k" V 2257 2551 50  0000 C CNN
 F 2 "" V 2180 2550 30  0001 C CNN
 F 3 "" H 2250 2550 30  0000 C CNN
@@
 P 3000 2000
 F 0 "C2" H 3050 2100 50  0000 L CNN
-F 1 "22n" H 3050 1900 50  0000 L CNN
+F 1 "15n" H 3050 1900 50  0000 L CNN
 F 2 "" H 3038 1850 30  0001 C CNN
 F 3 "" H 3000 2000 60  0000 C CNN
@@
 P 3250 2300
 F 0 "R8" V 3330 2300 50  0000 C CNN
-F 1 "4.7k" V 3257 2301 50  0000 C CNN
+F 1 "3.9k" V 3257 2301 50  0000 C CNN
 F 2 "" V 3180 2300 30  0001 C CNN
 F 3 "" H 3250 2300 30  0000 C CNN
@@
 P 3450 2000
 F 0 "C4" H 3500 2100 50  0000 L CNN
-F 1 "33n" H 3500 1900 50  0000 L CNN
+F 1 "3.3n" H 3500 1900 50  0000 L CNN
 F 2 "" H 3488 1850 30  0001 C CNN
 F 3 "" H 3450 2000 60  0000 C CNN
@@
 P 4150 2450
 F 0 "R10" V 4230 2450 50  0000 C CNN
-F 1 "480k" V 4157 2451 50  0000 C CNN
+F 1 "660k" V 4157 2451 50  0000 C CNN
 F 2 "" V 4080 2450 30  0001 C CNN
 F 3 "" H 4150 2450 30  0000 C CNN
@@
 P 3950 2450
 F 0 "R9" V 4030 2450 50  0000 C CNN
-F 1 "480k" V 3957 2451 50  0000 C CNN
+F 1 "660k" V 3957 2451 50  0000 C CNN
 F 2 "" V 3880 2450 30  0001 C CNN
 F 3 "" H 3950 2450 30  0000 C CNN
@@
 P 4400 1550
 F 0 "R11" V 4480 1550 50  0000 C CNN
-F 1 "15k" V 4407 1551 50  0000 C CNN
+F 1 "8.2k" V 4407 1551 50  0000 C CNN
 F 2 "" V 4330 1550 30  0001 C CNN
 F 3 "" H 4400 1550 30  0000 C CNN
@@
 P 3900 2000
 F 0 "C5" H 3950 2100 50  0000 L CNN
-F 1 "33n" H 3950 1900 50  0000 L CNN
+F 1 "3.3n" H 3950 1900 50  0000 L CNN
 F 2 "" H 3938 1850 30  0001 C CNN
 F 3 "" H 3900 2000 60  0000 C CNN
@@
 P 5650 2000
 F 0 "R12" V 5730 2000 50  0000 C CNN
-F 1 "11k" V 5657 2001 50  0000 C CNN
+F 1 "8.2k" V 5657 2001 50  0000 C CNN
 F 2 "mylib:Resistor_Horizontal_Shop" V 5580 2000 30  0001 C CNN
 F 3 "" H 5650 2000 30  0000 C CNN
@@
 P 7200 1500
 F 0 "C8" H 7250 1600 50  0000 L CNN
-F 1 "10n" H 7250 1400 50  0000 L CNN
+F 1 "22n" H 7250 1400 50  0000 L CNN
 F 2 "" H 7238 1350 30  0001 C CNN
 F 3 "" H 7200 1500 60  0000 C CNN
@@
 P 5950 2250
 F 0 "C6" H 6000 2350 50  0000 L CNN
-F 1 "22n" H 6000 2150 50  0000 L CNN
+F 1 "47n" H 6000 2150 50  0000 L CNN
 F 2 "" H 5988 2100 30  0001 C CNN
 F 3 "" H 5950 2250 60  0000 C CNN
@@
 P 6200 2000
 F 0 "R13" V 6280 2000 50  0000 C CNN
-F 1 "120k" V 6207 2001 50  0000 C CNN
+F 1 "100k" V 6207 2001 50  0000 C CNN
 F 2 "" V 6130 2000 30  0001 C CNN
 F 3 "" H 6200 2000 30  0000 C CNN
@@
 P 6750 2000
 F 0 "R14" V 6830 2000 50  0000 C CNN
-F 1 "33k" V 6757 2001 50  0000 C CNN
+F 1 "27k" V 6757 2001 50  0000 C CNN
 F 2 "" V 6680 2000 30  0001 C CNN
 F 3 "" H 6750 2000 30  0000 C CNN
